File: Hardware/KiCAD/controles/controles.sch (KiCad schematic (older format))
At the start: 18 parts

Commit message: Release 1.0.5
Other:
- note added: "GPIO2 (led)"
- note removed: "GPIO16 (led)"
Changed lines of the file:
@@
 3.3v
 Text Notes 900  2850 0    60   ~ 0
-GPIO16 (led)
+GPIO2 (led)
 Text Notes 1300 2950 0    60   ~ 0
 ADC

Commit message: controle.pdf updated
Other:
- note added: "GPIO2 (optionnal led)"
- note removed: "GPIO2 (led)"
Changed lines of the file:
@@
 Text Notes 1300 2750 0    60   ~ 0
 3.3v
-Text Notes 900  2850 0    60   ~ 0
-GPIO2 (led)
+Text Notes 500  2850 0    60   ~ 0
+GPIO2 (optionnal led)
 Text Notes 1300 2950 0    60   ~ 0
 ADC
